Commit message: Modifify right hand to use multiple degrees of freedom

File: src/humanoid_description/urdf/humanoid.urdf.xacro (robot description, xacro)
@@ -1,10 +1,8 @@
 <?xml version="1.0"?>
 <robot name="simple_humanoid" xmlns:xacro="http://www.ros.org/wiki/xacro">
+  <xacro:include filename="$(find humanoid_description)/urdf/right_arm.xacro"/>
   <!-- Materiale -->
   <material name="green">
     <color rgba="0 1 0 1"/> <!-- verde -->
-  </material>
-  <material name="red">
-    <color rgba="1 0 0 1"/> <!-- roșu -->
   </material>
   <material name="blue">
@@ -35,6 +33,7 @@
     </collision>
     <inertial>
-      <mass value="3.0"/>
-      <inertia ixx="0.1" ixy="0" ixz="0" iyy="0.1" iyz="0" izz="0.1"/>
+       <mass value="10.0"/> <!-- Masa mai mare pentru stabilitate -->
+      <inertia ixx="0.3" ixy="0" ixz="0" iyy="0.3" iyz="0" izz="0.3"/>
+      <origin xyz="0 0 -0.1" rpy="0 0 0"/> <!-- Centru de masă MAI JOS -->
     </inertial>
   </link>
@@ -53,6 +52,7 @@
     </collision>
     <inertial>
-      <mass value="8.0"/>
-      <inertia ixx="0.1" ixy="0" ixz="0" iyy="0.1" iyz="0" izz="0.1"/>
+      <mass value="15.0"/> <!-- Masa mai mare pentru stabilitate -->
+      <inertia ixx="0.3" ixy="0" ixz="0" iyy="0.3" iyz="0" izz="0.3"/>
+      <origin xyz="0 0 -0.1" rpy="0 0 0"/> <!-- Centru de masă MAI JOS -->
     </inertial>
   </link>
@@ -99,5 +99,5 @@
     </collision>
     <inertial>
-      <mass value="1.5"/>
+      <mass value="155.5"/>
       <inertia ixx="0.01" ixy="0" ixz="0" iyy="0.01" iyz="0" izz="0.01"/>
     </inertial>
@@ -106,5 +106,5 @@
     <parent link="left_thigh"/>
     <child link="left_calf"/>
-    <origin xyz="0 0 -${thigh_z/2}" rpy="0 0 0"/>
+    <origin xyz="0 0 -${thigh_z}" rpy="0 0 0"/>
     <axis xyz="0 1 0"/>
     <limit lower="0" upper="2.0" effort="5" velocity="1.0"/>
@@ -146,5 +146,5 @@
     </collision>
     <inertial>
-      <mass value="1.5"/>
+      <mass value="155.5"/>
       <inertia ixx="0.01" ixy="0" ixz="0" iyy="0.01" iyz="0" izz="0.01"/>
     </inertial>
@@ -153,5 +153,5 @@
   <parent link="right_thigh"/>
   <child link="right_calf"/>
-  <origin xyz="0 0 -${thigh_z/2}" rpy="0 0 0"/>
+  <origin xyz="0 0 -${thigh_z}" rpy="0 0 0"/>
   <axis xyz="0 1 0"/>
   <limit lower="0" upper="2.0" effort="5" velocity="1.0"/>
@@ -213,56 +213,5 @@
 </joint>
   <!-- Braț drept -->
-  <link name="right_upper_arm">
-    <visual>
-      <geometry>
-        <cylinder length="${arm_z}" radius="0.03"/>
-      </geometry>
-      <material name="green"/>
-    </visual>
-    <collision>
-      <geometry>
-        <cylinder length="${arm_z}" radius="0.03"/>
-      </geometry>
-    </collision>
-    <inertial>
-      <mass value="1.0"/>
-      <inertia ixx="0.005" ixy="0" ixz="0" iyy="0.005" iyz="0" izz="0.005"/>
-    </inertial>
-  </link>
-  <joint name="right_shoulder" type="fixed">
-    <parent link="torso"/>
-    <child link="right_upper_arm"/>
-    <origin xyz="${torso_x-0.1} 0 ${torso_z-0.33}" rpy="0 -0.14 -0.05"/>
-    <!-- <origin xyz="${torso_x/2} 0 ${torso_z/3}" rpy="0 0 0"/> -->
-  </joint>
-  <link name="right_forearm">
-    <visual>
-      <!-- mutăm cilindrul astfel încât să pornească din cot -->
-      <origin xyz="0 0 -${arm_z/2}" rpy="0 0 0"/>
-      <geometry>
-        <cylinder length="${arm_z}" radius="0.025"/>
-      </geometry>
-      <material name="green"/>
-    </visual>
-    <collision>
-      <!-- și pentru coliziune la fel -->
-      <origin xyz="0 0 -${arm_z/2}" rpy="0 0 0"/>
-      <geometry>
-        <cylinder length="${arm_z}" radius="0.025"/>
-      </geometry>
-    </collision>
-    <inertial>
-      <mass value="0.8"/>
-      <inertia ixx="0.4" ixy="0" ixz="0" iyy="0.4" iyz="0" izz="0.4"/>
-    </inertial>
-  </link>
-  <joint name="right_elbow" type="revolute">
-    <parent link="right_upper_arm"/>
-    <child link="right_forearm"/>
-    <!-- cotul la capătul inferior al brațului superior -->
-    <origin xyz="0 0 -${arm_z/2}" rpy="0 0 0"/>
-    <axis xyz="1 0 0"/>
-    <limit lower="0" upper="2.0" effort="3" velocity="1.0"/>
-  </joint>
+  <xacro:right_arm parent_link="torso"/>
   <!-- CAP -->
   <link name="head">
@@ -271,5 +220,4 @@
         <sphere radius="0.1"/>
       </geometry>
-      <material name="yellow"/>
     </visual>
     <collision>
